File: hw/EE445L_Lab_7_Starter.sch (EAGLE design)
At the start: 18 parts, among them Q1 IRLD024

Commit message: final Lab07 commit
Parts:
- removed D1: 1N914DO35-7, EE445L:1N914DO35-7
- removed DOWN, LEFT, MODE, RIGHT, UP: (no value), EE445L:B3F-1052
- removed Q1: IRLD024, EE445L:IRLD024
- removed SP1: SPEAKER, EE445L:SPEAKER
- removed TESTPOINT: TP_LOOP, EE445L:TP_LOOP
- added 3.3V, 5.0V, GND: TP_LOOP, EE445L:TP_LOOP
- added C3, C5: 4.7uf, EE445L:CAPACITOR_POLARIZEDE5-6
- added IC2: LM4041CILPRCLP, EE445L:LM4041CILPRCLP
- added IC3: MC34119P, EE445L:MC34119P
- added J1: 105017-0001, 105017-0001:105017-0001
- added JP1: (no value), EE445L:PINHD-1X2
- added LED2: (no value), EE445L:LED3MM
- added R1: 1K, EE445L:RESISTOR0204/5
- added U$5: POWER_CONN, EE445L:POWER_CONN
- added U$6: SW_POWER_100MIL, EE445L:SW_POWER_100MIL
- added U$7: LM2937-4PIN, EE445L:LM2937-4PIN
- U$4: value 2.1MM_BARREL_JACK -> TLV5618; device EE445L:2.1MM_BARREL_JACK -> EE445L:TLV5618
Connections:
- removed net DOWN: DOWN.S, DOWN.S1, U$2G$3.PC7
- removed net LEFT: LEFT.S, LEFT.S1, U$2G$3.PC6
- removed net MODE: MODE.S, MODE.S1, U$2G$6.PF4
- removed net N$1: D1.A, Q1.D, SP1.2
- removed net N$2: C1.+, C19.2, R3.2, U$1.4-CH_EN, U$1.8-VDD, U$4.VDD
- removed net RIGHT: RIGHT.S, RIGHT.S1, U$2G$3.PC5
- removed net UP: U$2G$3.PC4, UP.S, UP.S1
- new net LAUNCH_PAD_SW1: U$2G$6.PF4
- new net LED_POWER: LED2.A, R1.1
- new net PC4: U$2G$3.PC4
- new net PC5: U$2G$3.PC5
- new net PC6: U$2G$3.PC6
- new net PC7: U$2G$3.PC7
- new net POWER_INPUT: J1.VDD, U$5.VDD, U$6.P$1
- new net POWER_SWITCHED: JP1.1, U$6.P$2
- net +3V3: now also 3.3V.TP, C1.+, C19.2, C5.+, R1.2, R3.2, U$1.4-CH_EN, U$1.8-VDD, U$7.VO; no longer D1.C, SP1.1
- net +5V: now also 5.0V.TP, C3.+, JP1.2, U$7.VI; no longer U$2G$7.+5.0V
- net GND: now also C3.-, C5.-, GND.TP, J1.GND, LED2.C, U$5.GND, U$7.GND, U$7.PAD; no longer DOWN.P, DOWN.P1, LEFT.P, LEFT.P1, MODE.P, MODE.P1, Q1.S, RIGHT.P, RIGHT.P1, U$4.GND, UP.P, UP.P1
- net PB1: no longer Q1.G
Other:
- note added: "Be very careful here: 1) Do not connect two 3.3V regular outputs together, even if one regulator has no input voltage, The jumper on the LaunchPad should probably be removed 2) Do not connect a battery or other voltage supply to USB 5V pin to laptop"
- note added: "Remove R9 and R10 from LaunchPad to use both PB7 and PD1 and PB6 and PD0"
- note added: "Use this jumper to measure current"
- note added: "YOUR NAMES HERE"
- note removed: "C"
- note removed: "NOTE: ESP8266 requires a separate supply"
- note removed: "NOTE: Remove R9 R10, so PB7 is no longer connected to PD1, and PB6 is no longer connected to PD0"
- note removed: "September 7, 2021"
- note removed: "University of Texas Mark McDermott & Jonathan Valvano"
